File: FlowerManager.kicad_pcb (KiCad board)
At the start: 2 copper layers, 99.2 x 78 mm, 115 parts, among them J1 USB_B_Mini, J10 Conn_01x02_Male, J11 Conn_01x02_Male, J12 Conn_01x02_Male, J2 AVR-ISP-6, J3 Conn_01x03_Male, J4 Conn_01x02_Male, J8 Conn_01x02_Male, J9 Conn_01x02_Male, Q1 AO3406, Q2 AO3406, Q3 AO3406, Q4 AO3406, Q5 AO3406, Q6 AO3406, Q8 IRLML6402, Q9 AO3406, SW1 SW_Push, SW2 SW_Push, SW3 SW_Push, SW4 SW_Push, U1 ATmega324PA-AU, U10 74LVC1G08, U11 74LVC1G08, U12 74LVC1G08, U13 LP2985-3.3, U14 FT232RL, U2 DS1307Z+, U3 DS18B20, U4 LM27313YMF, U5 BMP280, U6 74LVC1G08, U7 74LVC1G08, U8 74LVC1G08, U9 74LVC1G08, Y1 FC135, Y2 Resonator

Commit message: fixed library rescue problem in schematic
Connections:
- DS1 pad 10: (no net) -> Net-(DS1-Pad10)
- DS1 pad 7: (no net) -> Net-(DS1-Pad7)
- DS1 pad 8: (no net) -> Net-(DS1-Pad8)
- DS1 pad 9: (no net) -> Net-(DS1-Pad9)
- J1 pad 4: (no net) -> Net-(J1-Pad4)
- U1 pad 25: (no net) -> Net-(U1-Pad25)
- U1 pad 30: (no net) -> Net-(U1-Pad30)
- U14 pad 10: (no net) -> Net-(U14-Pad10)
- U14 pad 11: (no net) -> Net-(U14-Pad11)
- U14 pad 12: (no net) -> Net-(U14-Pad12)
- U14 pad 13: (no net) -> Net-(U14-Pad13)
- U14 pad 19: (no net) -> Net-(U14-Pad19)
- U14 pad 2: (no net) -> Net-(U14-Pad2)
- U14 pad 22: (no net) -> Net-(U14-Pad22)
- U14 pad 27: (no net) -> Net-(U14-Pad27)
- U14 pad 28: (no net) -> Net-(U14-Pad28)
- U14 pad 3: (no net) -> Net-(U14-Pad3)
- U14 pad 6: (no net) -> Net-(U14-Pad6)
- U14 pad 9: (no net) -> Net-(U14-Pad9)
- U2 pad 7: (no net) -> Net-(U2-Pad7)
